Commit message: Add missing materials (bh_alone.urdf.xacro)

File: barrett_hand_description/robots/bh_alone.urdf.xacro (robot description, xacro)
@@ -3,4 +3,10 @@
 	<!-- Available choices: bh282.urdf.xacro, bh280.urdf.xacro -->
 	<xacro:include filename="$(find barrett_hand_description)/urdf/bh280.urdf.xacro" />
+	<material name="Blue">
+		<color rgba="0.0 0.0 0.8 1.0"/>
+	</material>
+	<material name="Green">
+		<color rgba="0.0 0.8 0.0 1.0"/>
+	</material>
 	<!-- z-coordinate is not 0 because otherwise the hand base tilts when the simulation is started -->
 	<link name="base_link">
